File: KiCad/VT100/VT100.kicad_pcb (KiCad board)
At the start: 2 copper layers, 22 parts, among them J1 Conn_01x04_Male, J2 USB_B, SW1 SW_Push, U1 AT89S52-24PC, U10 74LS573, U11 74LS573, U12 UM61256, U13 74LS573, U2 MC6845, U3 XC9536PC44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

Commit message: VT100 MCU, KiCad and CPLD
Parts:
- added J2: Conn_02x05_Odd_Even, Connector_PinHeader_2.54mm:PinHeader_2x05_P2.54mm_Vertical, F.Cu at (149.9, 53.3)
- added J4: DB15_Female_HighDensity_MountingHoles, Connector_Dsub:DSUB-15-HD_Female_Horizontal_P2.29x1.98mm_EdgePinOffset3.03mm_Housed_MountingHolesOffset4.94mm, F.Cu at (201.9, 109.2)
- added R2: 1K, Resistor_THT:R_Axial_DIN0204_L3.6mm_D1.6mm_P1.90mm_Vertical, F.Cu at (215.3, 134.7)
- added R3: 1K, Resistor_THT:R_Axial_DIN0204_L3.6mm_D1.6mm_P1.90mm_Vertical, F.Cu at (187.7, 152.2)
- added R4: 1K, Resistor_THT:R_Axial_DIN0204_L3.6mm_D1.6mm_P1.90mm_Vertical, F.Cu at (182.7, 152.2)
- added R5: 1K, Resistor_THT:R_Axial_DIN0204_L3.6mm_D1.6mm_P1.90mm_Vertical, F.Cu at (237.4, 107.7)
- added U11: 74LS573 Char, Package_DIP:DIP-20_W7.62mm, F.Cu at (193.6, 125.7)
- added U15: 74LS573 Color Buffer, Package_DIP:DIP-20_W7.62mm, F.Cu at (261.0, 74.9)
- added U16: 74LS573 Charline, Package_DIP:DIP-20_W7.62mm, F.Cu at (204.5, 125.7)
- added U17: 74LS299, Package_DIP:DIP-20_W7.62mm, F.Cu at (215.7, 108.2)
- added U18: 74LS573 Color, Package_DIP:DIP-20_W7.62mm, F.Cu at (182.8, 125.7)
- added U19: 74LS257, Package_DIP:DIP-16_W7.62mm, F.Cu at (226.6, 108.2)
- C2: renamed from C1; value C_Polarized_Small -> C_Pol.
- U10: value 74LS573 -> 74LS573 GA8-15
- U12: renamed from U11; value 74LS573 -> 74LS573 GD0-7
- U13: value 74LS573 -> 74LS573 GD0-7
- U8: value 74LS245 -> 74LS245 CharsetAdr 1
- U9: value 74LS573 -> 74LS573 GA0-7
- moved R1 250.0 mm to (29.2, 114.3), turned to 0 degrees
- moved C2 249.5 mm to (38.1, 120.7), turned to 90 degrees
- moved C1 243.9 mm to (34.3, 106.7)
- moved C3 242.4 mm to (29.2, 106.7)
- moved SW1 241.2 mm to (26.7, 120.7)
- moved Crystal1 231.2 mm to (34.3, 101.6), turned to 180 degrees
- moved J1 231.2 mm to (33.0, 41.1), turned to 90 degrees
- moved U7 181.6 mm to (57.1, 47.0)
- moved U4 179.1 mm to (45.7, 47.0)
- moved U1 177.9 mm to (27.9, 47.0)
- moved J3 174.5 mm to (45.7, 120.7), turned to 90 degrees
- moved U10 138.5 mm to (78.7, 82.5)
- moved U13 135.4 mm to (78.8, 29.2)
- moved X1 123.3 mm to (101.6, 119.4)
- moved U9 118.2 mm to (78.7, 55.9)
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- renumbered C2 to C1, J2 to J1, J1 to J3, U12 to U14
Connections:
- U1 pad 12: /P3.2 -> Charset
- U1 pad 13: /P3.3 -> Screen
- U1 pad 17: /P3.7 -> RD\
- U10 pad 12: unconnected-(U10-Pad12) -> Net-(U10-Pad12)
- U10 pad 9: unconnected-(U10-Pad9) -> T0
- U12 pad 1: OE_DATA -> GWE\
- U13 pad 1: CHAROE -> Net-(U10-Pad12)
- U13 pad 11: LOADCHR -> LOADDAT
- U13 pad 12: /GA11 -> /P1.7
- U13 pad 13: /GA10 -> /P1.6
- U13 pad 14: /GA9 -> /P1.5
- U13 pad 15: /GA8 -> /P1.4
- U13 pad 16: /GA7 -> /P1.3
- U13 pad 17: /GA6 -> /P1.2
- U13 pad 18: /GA5 -> /P1.1
- U13 pad 19: /GA4 -> /P1.0
- U2 pad 3: unconnected-(U2-Pad3) -> GND
- U3 pad 1: unconnected-(U3-Pad1) -> HSYNC
- U3 pad 14: PixClk*2 -> LoadSr
- U3 pad 15: unconnected-(U3-Pad15) -> TDI
- U3 pad 16: unconnected-(U3-Pad16) -> TMS
- U3 pad 17: unconnected-(U3-Pad17) -> TCK
- U3 pad 24: unconnected-(U3-Pad24) -> COLOR
- U3 pad 30: unconnected-(U3-Pad30) -> TDO
- U3 pad 4: /P3.7 -> unconnected-(U3-Pad4)
- U3 pad 40: unconnected-(U3-Pad40) -> LoadSr
- U3 pad 42: unconnected-(U3-Pad42) -> LoadCharline
- U3 pad 43: unconnected-(U3-Pad43) -> PixClkO
- U3 pad 44: unconnected-(U3-Pad44) -> VSYNC
- U3 pad 6: unconnected-(U3-Pad6) -> LOADDAT
- U3 pad 7: unconnected-(U3-Pad7) -> LoadCol
- U6 pad 7: /MA12 -> GND
- U6 pad 8: /MA13 -> Screen
- U8 pad 12: unconnected-(U8-Pad12) -> /GA14
- U8 pad 13: unconnected-(U8-Pad13) -> /GA13
- U8 pad 14: unconnected-(U8-Pad14) -> /GA12
- U8 pad 19: unconnected-(U8-Pad19) -> CHAROE
- U8 pad 6: unconnected-(U8-Pad6) -> Charset
- U8 pad 7: unconnected-(U8-Pad7) -> +5V
- U8 pad 8: unconnected-(U8-Pad8) -> Screen
Other:
- board outline added: 99.1 x 99.1 mm
