File: KiCad/VT100/VT100.kicad_sch (KiCad schematic)
At the start: 22 parts, among them J1 Conn_01x04_Male, J2 USB_B, SW1 SW_Push, U1 AT89S52-24PC, U10 74LS573, U11 74LS573, U12 UM61256, U13 74LS573, U2 MC6845, U3 XC9536PC44, U4 74LS573, U5 74LS245, U6 74LS245, U7 UM61256, U8 74LS245, U9 74LS573, X1 25.175Mhz

Commit message: VT100 MCU, KiCad and CPLD
Parts:
- added J2: Conn_02x05_Odd_Even, Connector_PinHeader_2.54mm:PinHeader_2x05_P2.54mm_Vertical, symbol Connector_Generic:Conn_02x05_Odd_Even
- added J4: DB15_Female_HighDensity_MountingHoles, Connector_Dsub:DSUB-15-HD_Female_Horizontal_P2.29x1.98mm_EdgePinOffset3.03mm_Housed_MountingHolesOffset4.94mm, symbol Connector:DB15_Female_HighDensity_MountingHoles
- added R2, R3, R4, R5: 1K, Resistor_THT:R_Axial_DIN0204_L3.6mm_D1.6mm_P1.90mm_Vertical, symbol Device:R_Small
- added U11: 74LS573 Char, Package_DIP:DIP-20_W7.62mm, symbol 74xx:74LS573
- added U15: 74LS573 Color Buffer, Package_DIP:DIP-20_W7.62mm, symbol 74xx:74LS573
- added U16: 74LS573 Charline, Package_DIP:DIP-20_W7.62mm, symbol 74xx:74LS573
- added U17: 74LS299, Package_DIP:DIP-20_W7.62mm, symbol 74xx:74LS299
- added U18: 74LS573 Color, Package_DIP:DIP-20_W7.62mm, symbol 74xx:74LS573
- added U19: 74LS257, Package_DIP:DIP-16_W7.62mm, symbol 74xx_IEEE:74LS257
- C2: renamed from C1; value C_Polarized_Small -> C_Pol.
- U10: value 74LS573 -> 74LS573 GA8-15
- U12: renamed from U11; value 74LS573 -> 74LS573 GD0-7
- U13: value 74LS573 -> 74LS573 GD0-7
- U14: renamed from U12; value UM61256 -> UM61256 GraphRam
- U5: value 74LS245 -> 74LS245 CharColor Lo
- U6: value 74LS245 -> 74LS245 Char Color Hi
- U8: value 74LS245 -> 74LS245 CharsetAdr 1
- U9: value 74LS573 -> 74LS573 GA0-7
- renumbered C2 to C1, J2 to J1, J1 to J3
Connections:
- net OE_DATA is gone; now on net GWE\: U12.1 (OE)
- net P3.2 is gone; now on net Charset: U1.12 (P3.2(*INT0))
- net P3.3 is gone; now on net Screen: U1.13 (P3.3(*INT1))
- net PixClk*2 is gone; now on net LoadSr: U3.14 (M12)
- net +5V: now also U8.7 (A5), J2.4 (Pin_4), U11.20 (VCC), U15.20 (VCC), U16.20 (VCC), U17.19 (S1), U17.2 (OE1), U17.20 (VCC), U17.3 (OE2), U17.9 (Mr), U18.20 (VCC), U19.16 (VCC)
- net CHAROE: now also U8.19 (CE), U11.1 (OE); no longer U13.1 (OE)
- net COLOR: now also U3.24 (M17)
- net GA10: now also U11.13 (Q6); no longer U13.13 (Q6)
- net GA11: now also U11.12 (Q7); no longer U13.12 (Q7)
- net GA12: now also U8.14 (B4)
- net GA13: now also U8.13 (B5)
- net GA14: now also U8.12 (B6)
- net GA4: now also U11.19 (Q0); no longer U13.19 (Q0)
- net GA5: now also U11.18 (Q1); no longer U13.18 (Q1)
- net GA6: now also U11.17 (Q2); no longer U13.17 (Q2)
- net GA7: now also U11.16 (Q3); no longer U13.16 (Q3)
- net GA8: now also U11.15 (Q4); no longer U13.15 (Q4)
- net GA9: now also U11.14 (Q5); no longer U13.14 (Q5)
- net GD0: now also U11.2 (D0), U15.2 (D0), U16.2 (D0)
- net GD1: now also U11.3 (D1), U15.3 (D1), U16.3 (D1)
- net GD2: now also U11.4 (D2), U15.4 (D2), U16.4 (D2)
- net GD3: now also U11.5 (D3), U15.5 (D3), U16.5 (D3)
- net GD4: now also U11.6 (D4), U15.6 (D4), U16.6 (D4)
- net GD5: now also U11.7 (D5), U15.7 (D5), U16.7 (D5)
- net GD6: now also U11.8 (D6), U15.8 (D6), U16.8 (D6)
- net GD7: now also U11.9 (D7), U15.9 (D7), U16.9 (D7)
- net GND: now also U2.3 (LPSTB), U6.7 (A5), J2.10 (Pin_10), J2.2 (Pin_2), J4.10, J4.5, J4.6, J4.7, J4.8, U11.10 (GND), U15.1 (OE), U15.10 (GND), U16.1 (OE), U16.10 (GND), U17.10 (GND), U18.1 (OE), U18.10 (GND), U19.8 (GND)
- net LOADCHR: now also U11.11 (Load); no longer U13.11 (Load)
- net MA12: no longer U6.7 (A5)
- net MA13: no longer U6.8 (A6)
- net P1.0: now also U13.19 (Q0)
- net P1.1: now also U13.18 (Q1)
- net P1.2: now also U13.17 (Q2)
- net P1.3: now also U13.16 (Q3)
- net P1.4: now also U13.15 (Q4)
- net P1.5: now also U13.14 (Q5)
- net P1.6: now also U13.13 (Q6)
- net P1.7: now also U13.12 (Q7)
- net RD\: now also U1.17 (P3.7(*RD))
- net T0: now also U10.9 (D7)
- net HSYNC: now reaches U3.1 (M1)
- net HSYNC: now also J4.13
- net TDI: now reaches U3.15 (TDI)
- net TDI: now also J2.9 (Pin_9)
- net TMS: now reaches U3.16 (TMS)
- net TMS: now also J2.5 (Pin_5)
- net TCK: now reaches U3.17 (TCK)
- net TCK: now also J2.1 (Pin_1)
- net TDO: now reaches U3.30 (TDO)
- net TDO: now also J2.3 (Pin_3)
- net LoadSr: now reaches U3.40 (I/O/GTS2)
- net LoadSr: now also U17.1 (S0), U18.11 (Load)
- net LoadCharline: now reaches U3.42 (I/O/GTS1)
- net LoadCharline: now also U16.11 (Load)
- net PixClkO: now reaches U3.43 (M4)
- net PixClkO: now also U17.12 (Cp)
- net VSYNC: now reaches U3.44 (M2)
- net VSYNC: now also J4.14
- net LOADDAT: now reaches U3.6 (I/O/GCK2)
- net LOADDAT: now also U13.11 (Load)
- net LoadCol: now reaches U3.7 (I/O/GCK3)
- net LoadCol: now also U15.11 (Load)
- net at U10.12 (Q7): now also U13.1 (OE)
- net Charset: now reaches U8.6 (A4)
- net Screen: now reaches U8.8 (A6)
- net Screen: now also U6.8 (A6)
- net P3.7: no longer names the net of U3.4 (M4)
- net P3.7: no longer U1.17 (P3.7(*RD))
- new net: R4.1, U19.12 (Qc)
- new net: J4.3, R4.2
- new net: R2.1, U19.4 (Qa)
- new net: J4.1, R2.2
- new net: U17.8 (Q0), U19.1 (S)
- new net: R3.1, U19.7 (Qb)
- new net: R5.1, U19.9 (Qd)
- new net: J4.2, R3.2
- new net CBuf0: U18.19 (Q0), U19.2 (I0a)
- new net CBuf1: U18.18 (Q1), U19.5 (I0b)
- new net CBuf2: U18.17 (Q2), U19.14 (I0c)
- new net CBuf3: U18.16 (Q3), U19.11 (I0d)
- new net CBuf4: U18.15 (Q4), U19.3 (I1a)
- new net CBuf5: U18.14 (Q5), U19.6 (I1b)
- new net CBuf6: U18.13 (Q6), U19.13 (I1c)
- new net CBuf7: U18.12 (Q7), U19.10 (I1d)
- new net CL0: U16.19 (Q0), U17.16 (IO7)
- new net CL1: U16.18 (Q1), U17.4 (IO6)
- new net CL2: U16.17 (Q2), U17.15 (IO5)
- new net CL3: U16.16 (Q3), U17.5 (IO4)
- new net CL4: U16.15 (Q4), U17.14 (IO3)
- new net CL5: U16.14 (Q5), U17.6 (IO2)
- new net CL6: U16.13 (Q6), U17.13 (IO1)
- new net CL7: U16.12 (Q7), U17.7 (IO0)
- new net Col0: U15.19 (Q0), U18.2 (D0)
- new net Col1: U15.18 (Q1), U18.3 (D1)
- new net Col2: U15.17 (Q2), U18.4 (D2)
- new net Col3: U15.16 (Q3), U18.5 (D3)
- new net Col4: U15.15 (Q4), U18.6 (D4)
- new net Col5: U15.14 (Q5), U18.7 (D5)
- new net Col6: U15.13 (Q6), U18.8 (D6)
- new net Col7: U15.12 (Q7), U18.9 (D7)
- new net DispEn: U19.15 (~{EN})
Other:
- moved on the sheet: C2, J3, R1, SW1, U10, U12, U14, U2, U8, U9, X1
