File: KiCad/VT100/VT100_MCU/VT100_MCU.kicad_pcb (KiCad board)
At the start: 2 copper layers, 100.3 x 100.3 mm, 47 parts, among them J1 USB_B, J2 Conn_02x05_Odd_Even, J3 Conn_01x04_Male, J4 Conn_02x36_Odd_Even, SW1 SW_Push, U1 AT89S52-24PC, U2 74LS573, U3 XC9536PC44, U4 UM61256, U5 74LS573 GA0-7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

Commit message: mcu+graph
Parts:
- removed REF**: PinHeader_1x10_P2.54mm_Vertical, Connector_PinHeader_2.54mm:PinHeader_1x10_P2.54mm_Vertical
- removed REF** (x6): PinHeader_1x22_P2.54mm_Vertical, Connector_PinHeader_2.54mm:PinHeader_1x22_P2.54mm_Vertical
- removed REF**: PinHeader_1x05_P2.54mm_Vertical, Connector_PinHeader_2.54mm:PinHeader_1x05_P2.54mm_Vertical
- removed REF**: PinHeader_1x04_P2.54mm_Vertical, Connector_PinHeader_2.54mm:PinHeader_1x04_P2.54mm_Vertical
- removed REF** (x3): PinHeader_1x09_P2.54mm_Vertical, Connector_PinHeader_2.54mm:PinHeader_1x09_P2.54mm_Vertical
- removed REF**: PinHeader_1x02_P2.54mm_Vertical, Connector_PinHeader_2.54mm:PinHeader_1x02_P2.54mm_Vertical
- removed REF**: PinHeader_1x06_P2.54mm_Vertical, Connector_PinHeader_2.54mm:PinHeader_1x06_P2.54mm_Vertical
- removed REF**: PinHeader_1x07_P2.54mm_Vertical, Connector_PinHeader_2.54mm:PinHeader_1x07_P2.54mm_Vertical
- removed REF**: PinHeader_1x11_P2.54mm_Vertical, Connector_PinHeader_2.54mm:PinHeader_1x11_P2.54mm_Vertical
- removed REF**: PinHeader_1x12_P2.54mm_Vertical, Connector_PinHeader_2.54mm:PinHeader_1x12_P2.54mm_Vertical
- removed REF**: PinHeader_1x08_P2.54mm_Vertical, Connector_PinHeader_2.54mm:PinHeader_1x08_P2.54mm_Vertical
- removed REF**: PinHeader_1x01_P2.54mm_Vertical, Connector_PinHeader_2.54mm:PinHeader_1x01_P2.54mm_Vertical
- removed REF**: PinHeader_1x15_P2.54mm_Vertical, Connector_PinHeader_2.54mm:PinHeader_1x15_P2.54mm_Vertical
- removed REF**: PinHeader_1x13_P2.54mm_Vertical, Connector_PinHeader_2.54mm:PinHeader_1x13_P2.54mm_Vertical
- removed REF**: PinHeader_1x03_P2.54mm_Vertical, Connector_PinHeader_2.54mm:PinHeader_1x03_P2.54mm_Vertical
- moved U5 4.84 mm to (86.3, 88.3)
- moved U6 4.84 mm to (100.3, 68.6)
- moved U7 4.84 mm to (92.7, 86.4)
- moved U4 4.84 mm to (62.2, 63.5)
- moved C5 4.84 mm to (50.2, 31.1)
- moved C1 4.84 mm to (27.3, 39.4)
- moved C2 4.84 mm to (33.0, 24.1)
- moved C3 4.84 mm to (18.4, 39.4)
- moved Crystal1 4.84 mm to (25.4, 33.7)
- moved D1 4.84 mm to (14.6, 47.0)
- moved J1 4.84 mm to (19.7, 27.7)
- moved R1 4.84 mm to (38.1, 23.8)
- moved SW1 4.84 mm to (31.8, 15.9)
- moved U1 4.84 mm to (43.8, 35.6)
- moved C6 4.84 mm to (35.6, 29.2)
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Connections:
- net COLOR renamed DispEn
- J4 pad 10: unconnected-(J4-Pad10) -> Charset
- J4 pad 12: unconnected-(J4-Pad12) -> Screen
- J4 pad 6: unconnected-(J4-Pad6) -> T0
- J4 pad 62: /Dummy11 -> OE_ADR
- J4 pad 8: unconnected-(J4-Pad8) -> T1
- U3 pad 25: /Dummy11 -> OE_ADR
- U3 pad 4: unconnected-(U3-Pad4) -> RD\
Routing:
- net OE_ADR: track 54.3 -> 83.9 mm, vias 0 -> 2
- net /Dummy11: track 29.6 -> 0.00 mm, vias 2 -> 0
